File: hardware/ESP32 UWB v1.0.sch (EAGLE design)
At the start: 53 parts, among them IC1 CP2104, J2 HEADER-12P-2.54, J3 USB-MICRO-5P, Q3 S8050, Q4 S8050, U1 ESP32-WROVER, U2 ME6217C33M5G, U3 ESP-WROOM-32, U4 LD1117/3.3v, U5 DWM1000

Commit message: swaped ESP module to ESP32-C3-MINI
Parts:
- removed U1: ESP32-WROVER, ESP32-Wrover:ESP32-WROVER
- removed U3: ESP-WROOM-32, esp32:ESP-WROOM-32
- added U6: ESP32-C3-MINI-1-N4, ESP32-C3-MINI-1-N4:ESP32-C3-MINI-1-N4
Connections:
- removed net CLK: U1.CLK, U3.CLK
- removed net CMD: U1.CMD, U3.CMD
- removed net IO12/MISO: J1.P$6, R6.2, U1.IO12, U3.IO12
- removed net IO13/MOSI: J1.P$7, R16.2, U1.IO13, U3.IO13
- removed net IO14/SCLK: J1.P$8, R17.2, U1.IO14, U3.IO14
- removed net IO15/NSS: J1.P$9, R18.2, U1.IO15, U3.IO15
- removed net IO16: J2.8, U1.NC1, U3.IO16
- removed net IO17: J2.9, U1.NC2, U3.IO17
- removed net IO21/RES: J2.10, U1.IO21, U3.IO21
- removed net IO22/DC: J2.11, U1.IO22, U3.IO22
- removed net IO23: J2.12, U1.IO23, U3.IO23, U5.SPIMOSI
- removed net IO25: J1.P$12, U1.IO25, U3.IO25
- removed net IO26: J1.P$13, U1.IO26, U3.IO26
- removed net IO34: J1.P$17, R15.1, U1.IO34, U3.IO34, U5.IRQ
- removed net IO35: J1.P$18, U1.IO35, U3.IO35
- removed net IO36/SVP: J1.P$19, U1.SENSR_VP, U3.SENSOR_VP
- removed net IO39/SVN: J1.P$20, U1.SENSR_VN, U3.SENSOR_VN
- removed net IO4: J2.6, U1.IO4, U3.IO4, U5.SPICSN
- removed net IO5: J2.7, U1.IO5, U3.IO5
- removed net NC: U1.NC, U3.NC
- removed net SD0: U1.SD0, U3.SDO
- removed net SD1: U1.SD1, U3.SD1
- removed net SD2: U1.SD2, U3.SD2
- removed net SD3: U1.SD3, U3.SD3
- new net IO1: J1.P$7, U6.IO1
- new net IO10: J1.P$9, U6.IO10
- new net IO3: J1.P$5, U6.IO3
- new net IO4/MOSI: J2.12, R16.2, U5.SPIMOSI, U6.IO4
- new net IO5/MISO: J2.11, R6.2, U5.SPIMISO, U6.IO5
- new net IO6/SCLK: J2.10, R17.2, U5.SPICLK, U6.IO6
- new net IO7: J2.9, R15.1, U5.IRQ, U6.IO7
- new net IO8/CS: J2.8, R18.2, U5.SPICSN, U6.IO8
- new net IO9: J2.7, Q3.C, R10.2, R7.1, U6.IO9
- net +3V3: now also J1.P$10, J1.P$11, U6.3V3; no longer U1.3V3, U3.3V3
- net GND: now also J1.P$12, J1.P$13, J1.P$14, J1.P$15, J1.P$16, J1.P$17, J1.P$18, J1.P$19, J1.P$20, U6.GND; no longer U1.GND1, U1.GND2, U1.GND3, U1.P_GND, U3.GND, U3.GND@1, U3.GND@15, U3.GND@38
- net IO0: now also J1.P$8, U6.IO0; no longer J2.5, Q3.C, R10.2, R7.1, U1.IO0, U3.IO0
- net IO18: now also J2.6, U6.IO18; no longer J1.P$10, U1.IO18, U3.IO18, U5.SPICLK
- net IO19: now also J2.5, U6.IO19; no longer J1.P$11, U1.IO19, U3.IO19, U5.SPIMISO
- net IO2: now also J1.P$6, U6.IO2; no longer J1.P$5, U1.IO2, U3.IO2
- net IO27: no longer J1.P$14, U1.IO27, U3.IO27
- net IO32: no longer J1.P$15, U1.IO32, U3.IO32
- net IO33: no longer J1.P$16, U1.IO33, U3.IO33
- net RESET: now also U6.EN; no longer U1.EN, U3.EN
- net RXD: now also U6.RXD0; no longer U1.RXD0, U3.RXD0
- net TXD: now also U6.TXD0; no longer U1.TXD0, U3.TXD0
Other:
- note removed: "IO34~IO39 input only"
- note removed: "MTDI"
- moved on the sheet: C12, C4, FLASH, J1, R10, R7, R9
